Commit message: Updation of URDF

File: install/manipulator/share/manipulator/urdf/manipulator.urdf (robot description, URDF)
Before this commit: robot manipulator, 5 links, 4 joints
Links:
- removed link base_link
- added link link_0; visual cylinder length=0.1 radius=0.15
Joints:
- joint joint_12: limit lower=-1.57 upper=1.57 effort=10 velocity=1.0 -> lower=0 upper=1.571 effort=10 velocity=1.0; origin xyz=0 0 0.3 rpy=0 0 0 -> xyz=0 0 0.15 rpy=0 0 0
- joint joint_23: limit lower=-1.57 upper=1.57 effort=10 velocity=1.0 -> lower=0 upper=1.571 effort=10 velocity=1.0; origin xyz=0 0 0.3 rpy=0 0 0 -> xyz=0 0 0.15 rpy=0 0 0
- joint joint_34: limit lower=-1.57 upper=1.57 effort=10 velocity=1.0 -> lower=0 upper=1.571 effort=10 velocity=1.0; origin xyz=0 0 0.3 rpy=0 0 0 -> xyz=0 0 0.15 rpy=0 0 0
- joint joint_b1: limit lower=-1.57 upper=1.57 effort=10 velocity=1.0 -> (none); origin xyz=0 0 0.05 rpy=0 0 0 -> xyz=0 0 0.15 rpy=0 0 0; parent base_link -> link_0; type revolute -> continuous

Commit message: Updation of URDF

File: install/manipulator/share/manipulator/urdf/manipulator.urdf (robot description, URDF)
Before this commit: robot manipulator, 5 links, 4 joints
Joints:
- removed joint joint_b1
- added joint joint_01: type continuous, parent link_0, child link_1, origin xyz=0 0 0.15 rpy=0 0 0, axis 0 0 1

Commit message: URDF Update

File: install/manipulator/share/manipulator/urdf/manipulator.urdf (robot description, URDF)
Before this commit: robot manipulator, 5 links, 4 joints
Joints:
- joint joint_23: origin xyz=0 0 0.15 rpy=0 0 0 -> xyz=0 0 0.3 rpy=0 0 0
- joint joint_34: origin xyz=0 0 0.15 rpy=0 0 0 -> xyz=0 0 0.3 rpy=0 0 0

Commit message: URDF Updation

File: install/manipulator/share/manipulator/urdf/manipulator.urdf (robot description, URDF)
Before this commit: robot manipulator, 5 links, 4 joints
Links:
- added link link_5; visual cylinder length=0.3 radius=0.04
- added link link_6; visual sphere radius=0.05
- added link link_7; visual cylinder length=0.2 radius=0.04
- added link link_8; visual sphere radius=0.05
- link link_0: geometry visual cylinder length=0.1 radius=0.2
- link link_1: geometry visual cylinder length=0.4 radius=0.04
- link link_2: geometry visual sphere radius=0.05
- link link_3: geometry visual cylinder length=0.3 radius=0.04
- link link_4: geometry visual sphere radius=0.05
Joints:
- added joint joint_45: type revolute, parent link_4, child link_5, origin xyz=0 0 0.33 rpy=0 0 0, axis 0 1 0, limit lower=0 upper=1.571 effort=10 velocity=1.0
- added joint joint_56: type fixed, parent link_5, child link_6, origin xyz=0 0 0 rpy=0 0 0
- added joint joint_67: type revolute, parent link_6, child link_7, origin xyz=0 0 0.33 rpy=0 0 0, axis 0 1 0, limit lower=0 upper=1.571 effort=10 velocity=1.0
- added joint joint_78: type fixed, parent link_7, child link_8, origin xyz=0 0 0 rpy=0 0 0
- joint joint_01: origin xyz=0 0 0.15 rpy=0 0 0 -> xyz=0 0 0 rpy=0 0 0
- joint joint_12: axis 0 1 0 -> (none); limit lower=0 upper=1.571 effort=10 velocity=1.0 -> (none); origin xyz=0 0 0.15 rpy=0 0 0 -> xyz=0 0 0 rpy=0 0 0; type revolute -> fixed
- joint joint_23: origin xyz=0 0 0.3 rpy=0 0 0 -> xyz=0 0 0.43 rpy=0 0 0
- joint joint_34: axis 0 1 0 -> (none); limit lower=0 upper=1.571 effort=10 velocity=1.0 -> (none); origin xyz=0 0 0.3 rpy=0 0 0 -> xyz=0 0 0 rpy=0 0 0; type revolute -> fixed
